File: Knox's Hackpad:Fidget Toy V1 /PCB/hackpad.kicad_pcb (KiCad board)
At the start: 2 copper layers, 58.5 x 75.3 mm, 10 parts, among them J1 OLED DISPLAY, SW1 SW_Push, SW2 SW_Push, SW3 SW_Push, SW4 SW_Push, SW5 SW_Push, SW6 SW_Push, U1 XIAO-RP2040-DIP

Commit message: Add README
Parts:
- moved J1 39.8 mm to (126.2, 121.1), turned to 180 degrees
Routing:
- net GND: track 172.5 -> 202.9 mm
- net SDA: track 32.2 -> 13.4 mm
- net +5V: track 44.2 -> 28.6 mm
- net SCL: track 27.9 -> 17.0 mm
- net SW_4: track 46.0 -> 47.8 mm
- net SW_6: track 60.8 -> 62.0 mm, vias 1 -> 0
- net R_ESW: track 60.6 -> 61.2 mm
- net SW_5: vias 1 -> 0
Other:
- board text added: "SW6"
- board text added: "XIAO HERE!"
